Commit message: Inertia corrected + Mass Decreased

File: src/mybot_description/urdf/mybot.xacro (robot description, xacro)
@@ -7,5 +7,5 @@
     <pose>0 0 0.6 0 0 0</pose>
     <inertial>
-      <mass value="55.0"/>
+      <mass value="20.0"/>
       <origin xyz="0 0 0" rpy="0 0 0"/>
       <inertia
@@ -134,10 +134,10 @@
     <inertial>
       <origin xyz="0 0 0" rpy="0 1.5707 1.5707"/>
-      <mass value="8"/>
+      <mass value="10"/>
       <cylinder_inertia m="10" r="0.1" h="0.06"/>
       <inertia
-        ixx="1.0" ixy="0.0" ixz="0.0"
-        iyy="1.0" iyz="0.0"
-        izz="1.0"/>
+        ixx="0.028" ixy="0.0" ixz="0.0"
+        iyy="0.028" iyz="0.0"
+        izz="0.05"/>
     </inertial>
   </link>
@@ -158,10 +158,10 @@
     <inertial>
       <origin xyz="0 0 0" rpy="0 1.5707 1.5707"/>
-      <mass value="8"/>
+      <mass value="10"/>
       <cylinder_inertia m="10" r="0.1" h="0.06"/>
       <inertia
-        ixx="1.0" ixy="0.0" ixz="0.0"
-        iyy="1.0" iyz="0.0"
-        izz="1.0"/>
+        ixx="0.028" ixy="0.0" ixz="0.0"
+        iyy="0.028" iyz="0.0"
+        izz="0.05"/>
     </inertial>
   </link>

Commit message: Inertia Corrected + Multi-Robot Choice

File: src/mybot_description/urdf/mybot.xacro (robot description, xacro)
@@ -7,5 +7,15 @@
     <pose>0 0 0.6 0 0 0</pose>
     <inertial>
-      <mass value="20.0"/>
+      <mass value="35.0"/>
+      <origin xyz="0 0 0" rpy="0 0 0"/>
+      <inertia
+          ixx="2" ixy="0" ixz="0"
+          iyy="2.5" iyz="0"
+          izz="2"
+      />
+    </inertial>
+<!--
+    <inertial>
+      <mass value="65.0"/>
       <origin xyz="0 0 0" rpy="0 0 0"/>
       <inertia
@@ -15,4 +25,5 @@
       />
     </inertial>
+-->
     <collision name='collision'>
       <geometry>

Commit message: scaling Inertia to half

File: src/mybot_description/urdf/mybot.xacro (robot description, xacro)
@@ -7,13 +7,22 @@
     <pose>0 0 0.6 0 0 0</pose>
     <inertial>
+      <mass value="30.0"/>
+      <origin xyz="0 0 0" rpy="0 0 0"/>
+      <inertia
+          ixx="1.078" ixy="0" ixz="0"
+          iyy="2.09" iyz="0"
+          izz="2.61"
+      />
+    </inertial>
+<!--
+    <inertial>
       <mass value="35.0"/>
       <origin xyz="0 0 0" rpy="0 0 0"/>
       <inertia
-          ixx="2" ixy="0" ixz="0"
+          ixx="1.8" ixy="0" ixz="0"
           iyy="2.5" iyz="0"
           izz="2"
       />
     </inertial>
-<!--
     <inertial>
       <mass value="65.0"/>

Commit message: changes made for Simulation on Gazebo and Stage and Turtlesim

File: src/mybot_description/urdf/mybot.xacro (robot description, xacro)
@@ -4,5 +4,5 @@
   <xacro:include filename="$(find mybot_description)/urdf/materials.xacro" />
   <xacro:include filename="$(find mybot_description)/urdf/macros.xacro" />
-  <link name='chassis'>
+  <link name='base_link'>
     <pose>0 0 0.6 0 0 0</pose>
     <inertial>
@@ -189,5 +189,5 @@
     <origin xyz="0 0.25 -0.2" rpy="0 0 0"/>
     <child link="left_wheel"/>
-    <parent link="chassis"/>
+    <parent link="base_link"/>
     <axis xyz="0 1 0" rpy="0 0 0"/>
     <limit effort="100" velocity="100"/>
@@ -197,5 +197,5 @@
     <origin xyz="0 -0.25 -0.2" rpy="0 0 0"/>
     <child link="right_wheel"/>
-    <parent link="chassis"/>
+    <parent link="base_link"/>
     <axis xyz="0 1 0" rpy="0 0 0"/>
     <limit effort="100" velocity="100"/>
